File: main/main.sch (KiCad schematic (older format))
At the start: 22 parts, among them J1 VCC12V, J2 GND, J3 RX, J4 TX, J5 VCC5V, J6 OUTGND, J7 RX3V, J8 TX3V, Q1 BSS138, Q2 BSS138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

Commit message: update
Parts:
- removed C4: 100uF, Capacitor_Tantalum_SMD:CP_EIA-6032-28_Kemet-C_Pad2.25x2.35mm_HandSolder, symbol Device:CP
- removed U2: LD1117S33TR_SOT223, Package_TO_SOT_SMD:TO-252-2, symbol Regulator_Linear:LD1117S33TR_SOT223
- added C4: 0.1uF, Capacitor_SMD:C_0603_1608Metric_Pad1.05x0.95mm_HandSolder, symbol Device:C
- added C6: CP, Capacitor_SMD:CP_Elec_6.3x3, symbol Device:CP
- added C7: 47uF, Capacitor_SMD:C_0805_2012Metric_Pad1.15x1.40mm_HandSolder, symbol Device:C
- added C8: CP, Capacitor_Tantalum_SMD:CP_EIA-7343-30_AVX-N_Pad2.25x2.55mm_HandSolder, symbol Device:CP
- added U3: L78L33_SOT89, Package_TO_SOT_SMD:SOT-89-3, symbol Regulator_Linear:L78L33_SOT89
- C1: value 0.33uF -> 1uF; footprint Capacitor_THT:CP_Radial_D8.0mm_P3.50mm -> Capacitor_SMD:C_0603_1608Metric_Pad1.05x0.95mm_HandSolder
- C2: value 0.1uF -> 1uF; footprint Capacitor_SMD:C_0805_2012Metric_Pad1.15x1.40mm_HandSolder -> Capacitor_SMD:C_0603_1608Metric_Pad1.05x0.95mm_HandSolder
- C3: value 100uF -> CP; footprint Capacitor_Tantalum_SMD:CP_EIA-7360-38_Kemet-E_Pad2.25x4.25mm_HandSolder -> Capacitor_SMD:CP_Elec_6.3x3
- C5: footprint Capacitor_SMD:C_1206_3216Metric_Pad1.42x1.75mm_HandSolder -> Capacitor_SMD:C_0603_1608Metric_Pad1.05x0.95mm_HandSolder
- D1: footprint Diode_SMD:D_SMA-SMB_Universal_Handsoldering -> Diode_SMD:D_SMA
- U1: value L7805ABV-DG -> KIA7805API
Connections:
- net 3V3: now also C4.1, C8.1, U3.1 (OUT)
- net 5V: now also C5.1, C6.1, C7.1, U3.3 (IN); no longer C2.1, C3.1
- net GND: now also C4.2, C6.2, C7.2, C8.2, U3.2 (GND); no longer C1.2
- net VIN: now also C3.1; no longer C5.1
- net VCC12: now reaches D1.2 (A), J1.1 (Pin_1)
- net LV1 renamed LV1RX3V
- net LV2 renamed LV2TX3V
- new net: C1.2, C2.1
Other:
- note added: "2*50v=100vCap\n"
- note added: "3.3v TVS diode\nSMLVT3V3, Low Voltage Transil"
- note added: "5v OUT for HC-05"
- note added: "Protection resistors"
- note added: "RX 5v"
- note added: "STAG GBO BLUETOOTH \n with level shifter v2"
- note added: "TX5v"
- moved on the sheet: J1, J2, J3, J4, J6
